Commit message: Add: Spinning rotor visualization

File: phoenix_drone_simulation/envs/assets/cf21x_bullet.urdf (robot description, URDF)
Before this commit: robot cf21, 6 links, 5 joints
Links:
- link base_link: geometry collision cylinder length=.025 radius=.06; visual mesh filename=meshes/cf2withoutRotors.dae scale=0.87 0.87 0.87
- link m1_link: mass 0 -> 1.0e-9; geometry collision cylinder length=0.005 radius=0.015; visual mesh filename=meshes/propeller_ccw.dae scale=.022 .022 .022
- link m2_link: mass 0 -> 1.0e-9; geometry collision cylinder length=0.005 radius=0.015; visual mesh filename=meshes/propeller_cw.dae scale=.022 .022 .022
- link m3_link: mass 0 -> 1.0e-9; geometry collision cylinder length=0.005 radius=0.015; visual mesh filename=meshes/propeller_ccw.dae scale=.022 .022 .022
- link m4_link: mass 0 -> 1.0e-9; geometry collision cylinder length=0.005 radius=0.015; visual mesh filename=meshes/propeller_cw.dae scale=.022 .022 .022
Joints:
- removed joint prop0_joint
- added joint prop4_joint: type continuous, parent base_link, child m4_link, origin xyz=0.028 0.028 0.0108 rpy=0 0 0, axis 0 0 1
- joint center_of_mass_joint: axis (none) -> 0 0 1; type fixed -> continuous
- joint prop1_joint: axis (none) -> 0 0 -1; child m3_link -> m1_link; origin (none) -> xyz=0.028 -0.028 0.0108 rpy=0 0 0; type fixed -> continuous
- joint prop2_joint: axis (none) -> 0 0 1; origin (none) -> xyz=-0.028 -0.028 0.0108 rpy=0 0 0; type fixed -> continuous
- joint prop3_joint: axis (none) -> 0 0 -1; child m1_link -> m3_link; origin (none) -> xyz=-0.028 0.028 0.0108 rpy=0 0 0; type fixed -> continuous

Commit message: Add: original CF propeller files

File: phoenix_drone_simulation/envs/assets/cf21x_bullet.urdf (robot description, URDF)
Before this commit: robot cf21, 6 links, 5 joints
Links:
- link base_link: geometry collision cylinder length=.025 radius=.06; visual mesh filename=meshes/cf2withoutRotors.dae scale=0.86 0.86 0.86
- link m1_link: geometry collision cylinder length=0.005 radius=0.015; visual mesh filename=meshes/ccw_prop.stl scale=1 1 1
- link m2_link: geometry collision cylinder length=0.005 radius=0.015; visual mesh filename=meshes/cw_prop.stl scale=1 1 1
- link m3_link: geometry collision cylinder length=0.005 radius=0.015; visual mesh filename=meshes/ccw_prop.stl scale=1 1 1
- link m4_link: geometry collision cylinder length=0.005 radius=0.015; visual mesh filename=meshes/cw_prop.stl scale=1 1 1
